File: _autosave-ESP32_C3.kicad_sch (KiCad schematic)
At the start: 11 parts, among them J3 GSD090012SEU, U2 ESP32-C3-WROOM-02-H4, U4 CP2102N-Axx-xQFN20, U5 USBLC6-2SC6, U5 W25Q32JVSSIQ

Commit message: Done with most of the stuff. Pending: Flash Module
Parts:
- added C12, C7: 10u, symbol Device:C_Polarized
- added C13, C8: 0.1u, symbol Device:C
- added LED?: LTST-C170KGKT, LTST-C170KGKT:DIOC200X125X110, symbol LTST-C170KGKT:LTST-C170KGKT
- added LED?: LTST-C170TBKT, LTST-C170TBKT:DIOC200X125X110, symbol LTST-C170TBKT:LTST-C170TBKT
- added R15 (x2), R16: 50, symbol Device:R
- added R19: 10k, symbol Device:R
- added R? (x2): 470, symbol Device:R
Connections:
- net GND: now also C10.1, C9.2, J3.3 (VSS1), J3.6 (VSS2), J3.8 (DAT1), J3.9 (DAT2), J3.G1 (SHIELD_GND), J3.G2 (SHIELD_GND), J3.G3 (SHIELD_GND), J3.G4 (SHIELD_GND), U2.19 (GND), U2.20 (GND), U2.21 (GND), U2.22 (GND), U2.23 (GND), U2.24 (GND), U2.25 (GND), U2.26 (GND), U2.27 (GND), U2.28 (GND), U2.29 (GND), U2.30 (GND), U2.31 (GND), U2.32 (GND), U2.33 (GND), U2.34 (GND), U2.35 (GND), U2.36 (GND), U2.37 (GND), U2.38 (GND), U2.39 (GND), U2.9 (GND), C12.2, C13.1, C7.2, C8.1
- net +3.3V: now reaches C9.1
- net +3.3V: now also C10.2, J3.4 (VDD1), R11.1, U2.1 (3V3), U4.6 (VDD), U4.7 (VREGIN), C12.1, C13.2, C7.1, C8.2, LED?.+, LED?.+, R19.2
- net CD_SD: now reaches J3.1 (CD/DAT3)
- net CD_SD: now also U2.18 (IO0), R19.1
- net MOSI_DI: now reaches J3.2 (CMD)
- net MOSI_DI: now also R15.2
- net SCLK: now reaches J3.5 (CLK)
- net SCLK: now also R15.2
- net at J3.7 (DAT0): now also R16.1
- net at U4.19 (~{RXT}/GPIO.3): now also R?.1
- net at U4.20 (~{TXT}/GPIO.2): now also R?.2
- net CS: now reaches U2.10 (IO10)
- net TX_RX: now reaches U2.11 (RXD)
- net RX_TX: now reaches U2.12 (TXD)
- net GPIO_18: now reaches U2.13 (IO18)
- net GPIO_19: now reaches U2.14 (IO19)
- net SCL: now reaches U2.15 (IO3)
- net MISO_DO: now reaches U2.16 (IO2)
- net MISO_DO: now also R16.2
- net PHOTO_C: now reaches U2.17 (IO1)
- net EN: now reaches U2.2 (EN)
- net SDA: now reaches U2.3 (IO4)
- net MIC_OUT: now reaches U2.4 (IO5)
- net at U2.5 (IO6): now also R15.1
- net at U2.6 (IO7): now also R15.1
- net GPIO8: now reaches U2.7 (IO8)
- net BOOT: now reaches U2.8 (IO9)
- new net: LED?.-, R?.2
- new net: LED?.-, R?.1
- no-connect marks 0 -> 5
Other:
- note added: "ESP32-C3-02"
- note added: "USB MODULE"
- moved on the sheet: C10, C11, C9, J3, R11, R12, R13, U2, U4, U5
