File: ESP32_C3.kicad_sch (KiCad schematic)
At the start: 0 parts

Commit message: Done with flash module
Parts:
- added C10, C13, C14, C8: 0.1u, symbol Device:C
- added C11: 1u, symbol Device:C
- added C12, C7: 10u, symbol Device:C_Polarized
- added C9: 4.7u, symbol Device:C_Polarized
- added J3: GSD090012SEU, GSD090012SEU:AMPHENOL_GSD090012SEU, symbol GSD090012SEU:GSD090012SEU
- added LED?: LTST-C170KGKT, LTST-C170KGKT:DIOC200X125X110, symbol LTST-C170KGKT:LTST-C170KGKT
- added LED?: LTST-C170TBKT, LTST-C170TBKT:DIOC200X125X110, symbol LTST-C170TBKT:LTST-C170TBKT
- added R11: 1k, symbol Device:R
- added R12, R13: 475k, symbol Device:R
- added R15 (x2), R16, R22: 50, symbol Device:R
- added R19: 10k, symbol Device:R
- added R? (x2): 470, symbol Device:R
- added U2: ESP32-C3-WROOM-02-H4, ESP32-C3-WROOM-02-H4:MODULE_ESP32-C3-WROOM-02-H4, symbol ESP32-C3-WROOM-02-H4:ESP32-C3-WROOM-02-H4
- added U4: CP2102N-Axx-xQFN20, Package_DFN_QFN:SiliconLabs_QFN-20-1EP_3x3mm_P0.5mm, symbol Interface_USB:CP2102N-Axx-xQFN20
- added U5: W25Q32JVSSIQ, W25Q32JVSSIQ:SOIC127P790X216-8N, symbol W25Q32JVSSIQ:W25Q32JVSSIQ
- added U5: USBLC6-2SC6, Package_TO_SOT_SMD:SOT-23-6, symbol Power_Protection:USBLC6-2SC6
Connections:
- new net: C11.1, R12.2, R13.1, U4.8 (VBUS)
- new net: R22.2, U5.2 (DO(IO1))
- new net: J3.7 (DAT0), R16.1
- new net: LED?.-, R?.2
- new net: U4.12 (GND), U4.21 (GND), U4.3 (GND)
- new net: R?.1, U4.19 (~{RXT}/GPIO.3)
- new net: R?.2, U4.20 (~{TXT}/GPIO.2)
- new net: U4.4 (D+), U5.3 (I/O2)
- new net: U4.5 (D-), U5.1 (I/O1)
- new net: R11.2, U4.9 (~{RST})
- new net: LED?.-, R?.1
- new net: R15.1, U2.5 (IO6)
- new net: R15.1, U2.6 (IO7)
- new net +3.3V: C10.2, C12.1, C13.2, C14.1, C7.1, C8.2, C9.1, J3.4 (VDD1), LED?.+, LED?.+, R11.1, R19.2, U2.1 (3V3), U4.6 (VDD), U4.7 (VREGIN), U5.3 (~{WP}(IO2)), U5.7 (~{HOLD}/~{RESET}(IO3)), U5.8 (VCC)
- new net BOOT: U2.8 (IO9)
- new net CD_SD: J3.1 (CD/DAT3), R19.1, U2.18 (IO0)
- new net CS: U2.10 (IO10), U5.1 (~{CS})
- new net EN: U2.2 (EN)
- new net GND: C10.1, C11.2, C12.2, C13.1, C14.2, C7.2, C8.1, C9.2, J3.3 (VSS1), J3.6 (VSS2), J3.8 (DAT1), J3.9 (DAT2), J3.G1 (SHIELD_GND), J3.G2 (SHIELD_GND), J3.G3 (SHIELD_GND), J3.G4 (SHIELD_GND), R13.2, U2.19 (GND), U2.20 (GND), U2.21 (GND), U2.22 (GND), U2.23 (GND), U2.24 (GND), U2.25 (GND), U2.26 (GND), U2.27 (GND), U2.28 (GND), U2.29 (GND), U2.30 (GND), U2.31 (GND), U2.32 (GND), U2.33 (GND), U2.34 (GND), U2.35 (GND), U2.36 (GND), U2.37 (GND), U2.38 (GND), U2.39 (GND), U2.9 (GND), U5.2 (GND), U5.4 (GND)
- new net GPIO8: U2.7 (IO8)
- new net GPIO_18: U2.13 (IO18)
- new net GPIO_19: U2.14 (IO19)
- new net MIC_OUT: U2.4 (IO5)
- new net MISO_DO: R16.2, R22.1, U2.16 (IO2)
- new net MOSI_DI: J3.2 (CMD), R15.2, U5.5 (DI(IO0))
- new net PHOTO_C: U2.17 (IO1)
- new net RX_TX: U2.12 (TXD)
- new net SCL: U2.15 (IO3)
- new net SCLK: J3.5 (CLK), R15.2, U5.6 (CLK)
- new net SDA: U2.3 (IO4)
- new net TX_RX: U2.11 (RXD)
- new net USB_DN: U5.6 (I/O1)
- new net USB_DP: U5.4 (I/O2)
- new net VBUS: R12.1, U5.5 (VBUS)
- no-connect marks 0 -> 7
Other:
- note added: "ESP32-C3-02"
- note added: "Flask memory"
- note added: "SD-card MODULE"
- note added: "USB MODULE"
- note added: "USB_D+"
- note added: "USB_D-"
