File: esp32-sensorboard.kicad_sch (KiCad schematic)
At the start: 25 parts, among them J1 SS-52400-002, U1 MCP73871

Commit message: Done with flash module
Other:
- sheet ESP32_C3 ports: added USB_DN, USB_DP, VBUS; removed none
Changed lines of the file:
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@@
 	(wire
 		(pts
+			(xy 121.92 154.94) (xy 128.27 154.94)
+		)
+		(stroke
+			(width 0)
+			(type default)
+		)
+	)
+	(wire
+		(pts
 			(xy 179.07 88.9) (xy 186.69 88.9)
 		)
@@
 	(wire
 		(pts
+			(xy 121.92 170.18) (xy 129.54 170.18)
+		)
+		(stroke
+			(width 0)
+			(type default)
+		)
+	)
+	(wire
+		(pts
 			(xy 267.97 45.72) (xy 267.97 43.18)
 		)
@@
 		)
 	)
+	(wire
+		(pts
+			(xy 121.92 162.56) (xy 128.27 162.56)
+		)
+		(stroke
+			(width 0)
+			(type default)
+		)
+	)
 	(label "+5V_USB"
 		(at 179.07 92.71 0)
@@
 		)
 	)
+	(label "VBUS"
+		(at 129.54 170.18 0)
+		(effects
+			(font
+				(size 1.27 1.27)
+			)
+			(justify left bottom)
+		)
+	)
 	(label "+5V_USB"
 		(at 241.3 66.04 0)
@@
 		)
 	)
+	(label "USB_DP"
+		(at 128.27 162.56 0)
+		(effects
+			(font
+				(size 1.27 1.27)
+			)
+			(justify left bottom)
+		)
+	)
+	(label "USB_DN"
+		(at 128.27 154.94 0)
+		(effects
+			(font
+				(size 1.27 1.27)
+			)
+			(justify left bottom)
+		)
+	)
 	(label "USB_DN"
 		(at 81.28 40.64 0)
@@
 			)
 		)
+		(pin "USB_DN" input
+			(at 121.92 154.94 0)
+			(effects
+				(font
+					(size 1.27 1.27)
+				)
+				(justify right)
+			)
+		)
+		(pin "USB_DP" input
+			(at 121.92 162.56 0)
+			(effects
+				(font
+					(size 1.27 1.27)
+				)
+				(justify right)
+			)
+		)
+		(pin "VBUS" input
+			(at 121.92 170.18 0)
+			(effects
+				(font
+					(size 1.27 1.27)
+				)
+				(justify right)
+			)
+		)
